File: Hardware/KiCAD/LuminaryVer1/InputConnectors.sch (KiCad schematic (older format))
At the start: 7 parts, among them J1 10_Pin_JTAG, J10 ExtBattPwr, J12 USB_B_Micro, J2 Conn_01x06, U1 74HC14

Commit message: Removed GPIO output driver to increase versatility as IO. Added passive over-current/voltage protection.
Other:
- note added: "Schmitt triggered inputs to provide clean edges"
Changed lines of the file:
@@
 EESchema Schematic File Version 4
+LIBS:LuminaryVer1-cache
 EELAYER 29 0
 EELAYER END
@@
 Wire Wire Line
 	2950 3600 3050 3600
+Text Notes 4900 1750 0    50   ~ 0
+Schmitt triggered inputs to provide clean edges
 $EndSCHEMATC
