File: Hardware/KiCAD/LuminaryVer1/InputConnectors.sch (KiCad schematic (older format))
At the start: 13 parts, among them J1 JTAG, J10 ExtBattPwr, J12 USB_B_Micro, J2 GPIOInput, U1 74HC14

Commit message: Added majority of the logic level circuitry. Almost done routing connections.
Connections:
- net GPIO_INPUT_0: now also U1.6; no longer U1.2
- net GPIO_INPUT_2: now also U1.2; no longer U1.6
- net GPIO_INPUT_3: now also U1.12; no longer U1.8
- net GPIO_INPUT_5: now also U1.8; no longer U1.12
- net at J2.1 (Pin_1), R25.2: now also U1.5; no longer U1.1
- net at J2.3 (Pin_3), R23.2: now also U1.1; no longer U1.5
- net at J2.4 (Pin_4), R22.2: now also U1.13; no longer U1.9
- net at J2.6 (Pin_6), R20.2: now also U1.9; no longer U1.13
Other:
- moved on the sheet: U1A, U1C, U1D, U1F
Changed lines of the file:
@@
 L 74xx:74HC14 U1
 U 1 1 5E69C7F1
-P 5750 2150
-F 0 "U1" H 5750 2467 50  0000 C CNN
-F 1 "74HC14" H 5750 2376 50  0000 C CNN
-F 2 "Package_SO:TSSOP-14_4.4x5mm_P0.65mm" H 5750 2150 50  0001 C CNN
-F 3 "http://www.ti.com/lit/gpn/sn74HC14" H 5750 2150 50  0001 C CNN
-	1    5750 2150
+P 5750 3200
+F 0 "U1" H 5750 3517 50  0000 C CNN
+F 1 "74HC14" H 5750 3426 50  0000 C CNN
+F 2 "Package_SO:TSSOP-14_4.4x5mm_P0.65mm" H 5750 3200 50  0001 C CNN
+F 3 "http://www.ti.com/lit/gpn/sn74HC14" H 5750 3200 50  0001 C CNN
+	1    5750 3200
 	1    0    0    -1
 $EndComp
@@
 L 74xx:74HC14 U1
 U 3 1 5E69E21D
-P 5750 3200
-F 0 "U1" H 5750 3517 50  0000 C CNN
-F 1 "74HC14" H 5750 3426 50  0000 C CNN
-F 2 "Package_SO:TSSOP-14_4.4x5mm_P0.65mm" H 5750 3200 50  0001 C CNN
-F 3 "http://www.ti.com/lit/gpn/sn74HC14" H 5750 3200 50  0001 C CNN
-	3    5750 3200
+P 5750 2150
+F 0 "U1" H 5750 2467 50  0000 C CNN
+F 1 "74HC14" H 5750 2376 50  0000 C CNN
+F 2 "Package_SO:TSSOP-14_4.4x5mm_P0.65mm" H 5750 2150 50  0001 C CNN
+F 3 "http://www.ti.com/lit/gpn/sn74HC14" H 5750 2150 50  0001 C CNN
+	3    5750 2150
 	1    0    0    -1
 $EndComp
@@
 L 74xx:74HC14 U1
 U 4 1 5E69F536
-P 5750 3700
-F 0 "U1" H 5750 4017 50  0000 C CNN
-F 1 "74HC14" H 5750 3926 50  0000 C CNN
-F 2 "Package_SO:TSSOP-14_4.4x5mm_P0.65mm" H 5750 3700 50  0001 C CNN
-F 3 "http://www.ti.com/lit/gpn/sn74HC14" H 5750 3700 50  0001 C CNN
-	4    5750 3700
+P 5750 4700
+F 0 "U1" H 5750 5017 50  0000 C CNN
+F 1 "74HC14" H 5750 4926 50  0000 C CNN
+F 2 "Package_SO:TSSOP-14_4.4x5mm_P0.65mm" H 5750 4700 50  0001 C CNN
+F 3 "http://www.ti.com/lit/gpn/sn74HC14" H 5750 4700 50  0001 C CNN
+	4    5750 4700
 	1    0    0    -1
 $EndComp
@@
 L 74xx:74HC14 U1
 U 6 1 5E6A15AB
-P 5750 4700
-F 0 "U1" H 5750 5017 50  0000 C CNN
-F 1 "74HC14" H 5750 4926 50  0000 C CNN
-F 2 "Package_SO:TSSOP-14_4.4x5mm_P0.65mm" H 5750 4700 50  0001 C CNN
-F 3 "http://www.ti.com/lit/gpn/sn74HC14" H 5750 4700 50  0001 C CNN
-	6    5750 4700
+P 5750 3700
+F 0 "U1" H 5750 4017 50  0000 C CNN
+F 1 "74HC14" H 5750 3926 50  0000 C CNN
+F 2 "Package_SO:TSSOP-14_4.4x5mm_P0.65mm" H 5750 3700 50  0001 C CNN
+F 3 "http://www.ti.com/lit/gpn/sn74HC14" H 5750 3700 50  0001 C CNN
+	6    5750 3700
 	1    0    0    -1
 $EndComp

Commit message: Finalized for version 1 production.
Parts:
- C5: LCSC (none) -> C1525; PartNumber (none) -> CL05B104KO5NNNC
- J1: Digikey (none) -> 609-3712-ND; Mouser (none) -> 649-221111-00010T4LF
- J12: Digikey (none) -> H125718CT-ND; Mouser (none) -> 798-ZX62D-B-5PA830
- R20, R21, R22, R23, R24, R25: value 50k -> 47k; LCSC (none) -> C25792; PartNumber (none) -> 0402WGF4702TCE
- U1: LCSC (none) -> C5606; PartNumber (none) -> 74HC14PW,118
Changed lines of the file:
@@
 F 2 "Package_SO:TSSOP-14_4.4x5mm_P0.65mm" H 5750 3200 50  0001 C CNN
 F 3 "http://www.ti.com/lit/gpn/sn74HC14" H 5750 3200 50  0001 C CNN
+F 4 "C5606" H 5750 3200 50  0001 C CNN "LCSC"
+F 5 "74HC14PW,118" H 5750 3200 50  0001 C CNN "PartNumber"
 	1    5750 3200
 	1    0    0    -1
@@
 F 2 "Package_SO:TSSOP-14_4.4x5mm_P0.65mm" H 5750 2700 50  0001 C CNN
 F 3 "http://www.ti.com/lit/gpn/sn74HC14" H 5750 2700 50  0001 C CNN
+F 4 "C5606" H 5750 2700 50  0001 C CNN "LCSC"
+F 5 "74HC14PW,118" H 5750 2700 50  0001 C CNN "PartNumber"
 	2    5750 2700
 	1    0    0    -1
@@
 F 2 "Package_SO:TSSOP-14_4.4x5mm_P0.65mm" H 5750 2150 50  0001 C CNN
 F 3 "http://www.ti.com/lit/gpn/sn74HC14" H 5750 2150 50  0001 C CNN
+F 4 "C5606" H 5750 2150 50  0001 C CNN "LCSC"
+F 5 "74HC14PW,118" H 5750 2150 50  0001 C CNN "PartNumber"
 	3    5750 2150
 	1    0    0    -1
@@
 F 2 "Package_SO:TSSOP-14_4.4x5mm_P0.65mm" H 5750 4700 50  0001 C CNN
 F 3 "http://www.ti.com/lit/gpn/sn74HC14" H 5750 4700 50  0001 C CNN
+F 4 "C5606" H 5750 4700 50  0001 C CNN "LCSC"
+F 5 "74HC14PW,118" H 5750 4700 50  0001 C CNN "PartNumber"
 	4    5750 4700
 	1    0    0    -1
@@
 F 2 "Package_SO:TSSOP-14_4.4x5mm_P0.65mm" H 5750 4150 50  0001 C CNN
 F 3 "http://www.ti.com/lit/gpn/sn74HC14" H 5750 4150 50  0001 C CNN
+F 4 "C5606" H 5750 4150 50  0001 C CNN "LCSC"
+F 5 "74HC14PW,118" H 5750 4150 50  0001 C CNN "PartNumber"
 	5    5750 4150
 	1    0    0    -1
@@
 F 2 "Package_SO:TSSOP-14_4.4x5mm_P0.65mm" H 5750 3700 50  0001 C CNN
 F 3 "http://www.ti.com/lit/gpn/sn74HC14" H 5750 3700 50  0001 C CNN
+F 4 "C5606" H 5750 3700 50  0001 C CNN "LCSC"
+F 5 "74HC14PW,118" H 5750 3700 50  0001 C CNN "PartNumber"
 	6    5750 3700
 	1    0    0    -1
@@
 F 2 "Package_SO:TSSOP-14_4.4x5mm_P0.65mm" H 7700 3300 50  0001 C CNN
 F 3 "http://www.ti.com/lit/gpn/sn74HC14" H 7700 3300 50  0001 C CNN
+F 4 "C5606" H 7700 3300 50  0001 C CNN "LCSC"
+F 5 "74HC14PW,118" H 7700 3300 50  0001 C CNN "PartNumber"
 	7    7700 3300
 	1    0    0    -1
@@
 F 2 "Capacitor_SMD:C_0402_1005Metric" H 7300 3300 50  0001 C CNN
 F 3 "~" H 7300 3300 50  0001 C CNN
+F 4 "C1525" H 7300 3300 50  0001 C CNN "LCSC"
+F 5 "CL05B104KO5NNNC" H 7300 3300 50  0001 C CNN "PartNumber"
 	1    7300 3300
 	1    0    0    1
@@
 F 2 "USB:Amphenol-MicroB" H 2850 4550 50  0001 C CNN
 F 3 "~" H 2850 4550 50  0001 C CNN
+F 4 "798-ZX62D-B-5PA830" H 2700 4600 50  0001 C CNN "Mouser"
+F 5 "" H 2700 4600 50  0001 C CNN "PartNumber"
+F 6 "H125718CT-ND" H 2700 4600 50  0001 C CNN "Digikey"
 	1    2700 4600
 	1    0    0    -1
@@
 F 2 "Connector_PinHeader_1.27mm:PinHeader_2x05_P1.27mm_Vertical" H 2650 3400 50  0001 C CNN
 F 3 "~" H 2650 3400 50  0001 C CNN
+F 4 "649-221111-00010T4LF" H 2650 3400 50  0001 C CNN "Mouser"
+F 5 "" H 2650 3400 50  0001 C CNN "PartNumber"
+F 6 "609-3712-ND" H 2650 3400 50  0001 C CNN "Digikey"
 	1    2650 3400
 	1    0    0    -1
@@
 P 4900 2250
 F 0 "R25" H 4968 2296 50  0000 L CNN
-F 1 "50k" H 4968 2205 50  0000 L CNN
+F 1 "47k" H 4968 2205 50  0000 L CNN
 F 2 "Resistor_SMD:R_0402_1005Metric" V 4940 2240 50  0001 C CNN
 F 3 "~" H 4900 2250 50  0001 C CNN
+F 4 "C25792" H 4900 2250 50  0001 C CNN "LCSC"
+F 5 "0402WGF4702TCE" H 4900 2250 50  0001 C CNN "PartNumber"
 	1    4900 2250
 	1    0    0    -1
@@
 P 4650 2250
 F 0 "R23" H 4718 2296 50  0000 L CNN
-F 1 "50k" H 4718 2205 50  0000 L CNN
+F 1 "47k" H 4718 2205 50  0000 L CNN
 F 2 "Resistor_SMD:R_0402_1005Metric" V 4690 2240 50  0001 C CNN
 F 3 "~" H 4650 2250 50  0001 C CNN
+F 4 "C25792" H 4650 2250 50  0001 C CNN "LCSC"
+F 5 "0402WGF4702TCE" H 4650 2250 50  0001 C CNN "PartNumber"
 	1    4650 2250
 	1    0    0    -1
@@
 P 4400 2250
 F 0 "R21" H 4468 2296 50  0000 L CNN
-F 1 "50k" H 4468 2205 50  0000 L CNN
+F 1 "47k" H 4468 2205 50  0000 L CNN
 F 2 "Resistor_SMD:R_0402_1005Metric" V 4440 2240 50  0001 C CNN
 F 3 "~" H 4400 2250 50  0001 C CNN
+F 4 "C25792" H 4400 2250 50  0001 C CNN "LCSC"
+F 5 "0402WGF4702TCE" H 4400 2250 50  0001 C CNN "PartNumber"
 	1    4400 2250
 	1    0    0    -1
@@
 P 4550 1850
 F 0 "R22" H 4618 1896 50  0000 L CNN
-F 1 "50k" H 4618 1805 50  0000 L CNN
+F 1 "47k" H 4618 1805 50  0000 L CNN
 F 2 "Resistor_SMD:R_0402_1005Metric" V 4590 1840 50  0001 C CNN
 F 3 "~" H 4550 1850 50  0001 C CNN
+F 4 "C25792" H 4550 1850 50  0001 C CNN "LCSC"
+F 5 "0402WGF4702TCE" H 4550 1850 50  0001 C CNN "PartNumber"
 	1    4550 1850
 	1    0    0    -1
@@
 P 4800 1850
 F 0 "R24" H 4868 1896 50  0000 L CNN
-F 1 "50k" H 4868 1805 50  0000 L CNN
+F 1 "47k" H 4868 1805 50  0000 L CNN
 F 2 "Resistor_SMD:R_0402_1005Metric" V 4840 1840 50  0001 C CNN
 F 3 "~" H 4800 1850 50  0001 C CNN
+F 4 "C25792" H 4800 1850 50  0001 C CNN "LCSC"
+F 5 "0402WGF4702TCE" H 4800 1850 50  0001 C CNN "PartNumber"
 	1    4800 1850
 	1    0    0    -1
@@
 P 4300 1850
 F 0 "R20" H 4368 1896 50  0000 L CNN
-F 1 "50k" H 4368 1805 50  0000 L CNN
+F 1 "47k" H 4368 1805 50  0000 L CNN
 F 2 "Resistor_SMD:R_0402_1005Metric" V 4340 1840 50  0001 C CNN
 F 3 "~" H 4300 1850 50  0001 C CNN
+F 4 "C25792" H 4300 1850 50  0001 C CNN "LCSC"
+F 5 "0402WGF4702TCE" H 4300 1850 50  0001 C CNN "PartNumber"
 	1    4300 1850
 	1    0    0    -1
