File: Hardware/KiCAD/LuminaryVer1/LuminaryVer1.sch (KiCad schematic (older format))
At the start: 0 parts

Commit message: Added majority of the logic level circuitry. Almost done routing connections.
Connections:
- no-connect marks 0 -> 2
Changed lines of the file:
@@
 F12 "GPIO_0" B R 5800 2700 50
 F13 "GPIO_1" B R 5800 2800 50
-F14 "PWM_0" B R 5800 3000 50
-F15 "CAN_1_TX" B R 5800 3350 50
-F16 "CAN_1_RX" B R 5800 3450 50
-F17 "RS232_1_TX" B R 5800 5000 50
-F18 "RS232_1_RX" B R 5800 5100 50
-F19 "GPIO_2" B R 5800 2900 50
-F20 "SPI_1_MOSI" B R 5800 4200 50
-F21 "SPI_1_MISO" B R 5800 4300 50
-F22 "SPI_1_SCK" B R 5800 4400 50
-F23 "ADC_2" B R 5800 3800 50
-F24 "ADC_1" B R 5800 3700 50
-F25 "ADC_0" B R 5800 3600 50
-F26 "PWM_1" B R 5800 3100 50
-F27 "PWM_2" B R 5800 3200 50
-F28 "GPIO_IN_0" B L 4650 4250 50
-F29 "GPIO_IN_1" B L 4650 4350 50
-F30 "GPIO_IN_2" B L 4650 4450 50
-F31 "GPIO_IN_3" B L 4650 4550 50
-F32 "GPIO_IN_4" B L 4650 4650 50
-F33 "GPIO_IN_5" B L 4650 4750 50
+F14 "CAN_1_TX" B R 5800 3350 50
+F15 "CAN_1_RX" B R 5800 3450 50
+F16 "RS232_1_TX" B R 5800 5000 50
+F17 "RS232_1_RX" B R 5800 5100 50
+F18 "GPIO_2" B R 5800 2900 50
+F19 "SPI_1_MOSI" B R 5800 4200 50
+F20 "SPI_1_MISO" B R 5800 4300 50
+F21 "SPI_1_SCK" B R 5800 4400 50
+F22 "ADC_2" B R 5800 3800 50
+F23 "ADC_1" B R 5800 3700 50
+F24 "ADC_0" B R 5800 3600 50
+F25 "GPIO_IN_0" B L 4650 4250 50
+F26 "GPIO_IN_1" B L 4650 4350 50
+F27 "GPIO_IN_2" B L 4650 4450 50
+F28 "GPIO_IN_3" B L 4650 4550 50
+F29 "GPIO_IN_4" B L 4650 4650 50
+F30 "GPIO_IN_5" B L 4650 4750 50
+F31 "GPIO_3" B R 5800 3000 50
+F32 "GPIO_4" B R 5800 3100 50
+F33 "GPIO_5" B R 5800 3200 50
 $EndSheet
 $Sheet
@@
 	4600 2000 4450 2000
 Connection ~ 4450 2000
+NoConn ~ 4150 3100
+NoConn ~ 4150 3200
 $EndSCHEMATC
