File: Hardware/KiCAD/LuminaryVer1/OutputDrive.sch (KiCad schematic (older format))
At the start: 16 parts, among them U5 SN65HVD232

Commit message: Finalized for version 1 production.
Parts:
- C10: LCSC (none) -> C1525; PartNumber (none) -> CL05B104KO5NNNC
- D2, D3, D4, D5, D6, D7: value 3v3Zener -> 3.9V; LCSC (none) -> C353523; PartNumber (none) -> BZT52C3V9S
- R12: LCSC (none) -> C25079; PartNumber (none) -> 0402WGF1200TCE
- R14, R15, R16, R17, R18, R19: value 1.8k -> 2.0k; LCSC (none) -> C4109; PartNumber (none) -> 0402WGF2001TCE
- U5: LCSC (none) -> C30530; PartNumber (none) -> SN65HVD232DR
Changed lines of the file:
@@
 F 2 "Package_SO:SOIC-8_3.9x4.9mm_P1.27mm" H 1950 3000 50  0001 C CNN
 F 3 "http://www.ti.com/lit/ds/symlink/sn65hvd230.pdf" H 1850 3900 50  0001 C CNN
+F 4 "C30530" H 1950 3500 50  0001 C CNN "LCSC"
+F 5 "SN65HVD232DR" H 1950 3500 50  0001 C CNN "PartNumber"
 	1    1950 3500
 	1    0    0    -1
@@
 F 2 "Resistor_SMD:R_0402_1005Metric" V 2690 3540 50  0001 C CNN
 F 3 "~" H 2650 3550 50  0001 C CNN
+F 4 "C25079" H 2650 3550 50  0001 C CNN "LCSC"
+F 5 "0402WGF1200TCE" H 2650 3550 50  0001 C CNN "PartNumber"
 	1    2650 3550
 	1    0    0    -1
@@
 P 5600 2250
 F 0 "R14" V 5395 2250 50  0000 C CNN
-F 1 "1.8k" V 5486 2250 50  0000 C CNN
+F 1 "2.0k" V 5486 2250 50  0000 C CNN
 F 2 "Resistor_SMD:R_0402_1005Metric" V 5640 2240 50  0001 C CNN
 F 3 "~" H 5600 2250 50  0001 C CNN
+F 4 "C4109" H 5600 2250 50  0001 C CNN "LCSC"
+F 5 "0402WGF2001TCE" H 5600 2250 50  0001 C CNN "PartNumber"
 	1    5600 2250
 	0    1    1    0
@@
 P 5850 2450
 F 0 "D2" V 5804 2529 50  0000 L CNN
-F 1 "3v3Zener" V 5895 2529 50  0000 L CNN
+F 1 "3.9V" V 5895 2529 50  0000 L CNN
 F 2 "Diode_SMD:D_SOD-323" H 5850 2450 50  0001 C CNN
 F 3 "~" H 5850 2450 50  0001 C CNN
+F 4 "C353523" H 5850 2450 50  0001 C CNN "LCSC"
+F 5 "BZT52C3V9S" H 5850 2450 50  0001 C CNN "PartNumber"
 	1    5850 2450
 	0    1    1    0
@@
 P 5600 3150
 F 0 "R15" V 5395 3150 50  0000 C CNN
-F 1 "1.8k" V 5486 3150 50  0000 C CNN
+F 1 "2.0k" V 5486 3150 50  0000 C CNN
 F 2 "Resistor_SMD:R_0402_1005Metric" V 5640 3140 50  0001 C CNN
 F 3 "~" H 5600 3150 50  0001 C CNN
+F 4 "C4109" H 5600 3150 50  0001 C CNN "LCSC"
+F 5 "0402WGF2001TCE" H 5600 3150 50  0001 C CNN "PartNumber"
 	1    5600 3150
 	0    1    1    0
@@
 P 5850 3350
 F 0 "D3" V 5804 3429 50  0000 L CNN
-F 1 "3v3Zener" V 5895 3429 50  0000 L CNN
+F 1 "3.9V" V 5895 3429 50  0000 L CNN
 F 2 "Diode_SMD:D_SOD-323" H 5850 3350 50  0001 C CNN
 F 3 "~" H 5850 3350 50  0001 C CNN
+F 4 "C353523" H 5850 3350 50  0001 C CNN "LCSC"
+F 5 "BZT52C3V9S" H 5850 3350 50  0001 C CNN "PartNumber"
 	1    5850 3350
 	0    1    1    0
@@
 P 5600 4050
 F 0 "R16" V 5395 4050 50  0000 C CNN
-F 1 "1.8k" V 5486 4050 50  0000 C CNN
+F 1 "2.0k" V 5486 4050 50  0000 C CNN
 F 2 "Resistor_SMD:R_0402_1005Metric" V 5640 4040 50  0001 C CNN
 F 3 "~" H 5600 4050 50  0001 C CNN
+F 4 "C4109" H 5600 4050 50  0001 C CNN "LCSC"
+F 5 "0402WGF2001TCE" H 5600 4050 50  0001 C CNN "PartNumber"
 	1    5600 4050
 	0    1    1    0
@@
 P 5850 4250
 F 0 "D4" V 5804 4329 50  0000 L CNN
-F 1 "3v3Zener" V 5895 4329 50  0000 L CNN
+F 1 "3.9V" V 5895 4329 50  0000 L CNN
 F 2 "Diode_SMD:D_SOD-323" H 5850 4250 50  0001 C CNN
 F 3 "~" H 5850 4250 50  0001 C CNN
+F 4 "C353523" H 5850 4250 50  0001 C CNN "LCSC"
+F 5 "BZT52C3V9S" H 5850 4250 50  0001 C CNN "PartNumber"
 	1    5850 4250
 	0    1    1    0
@@
 P 7750 2250
 F 0 "R17" V 7545 2250 50  0000 C CNN
-F 1 "1.8k" V 7636 2250 50  0000 C CNN
+F 1 "2.0k" V 7636 2250 50  0000 C CNN
 F 2 "Resistor_SMD:R_0402_1005Metric" V 7790 2240 50  0001 C CNN
 F 3 "~" H 7750 2250 50  0001 C CNN
+F 4 "C4109" H 7750 2250 50  0001 C CNN "LCSC"
+F 5 "0402WGF2001TCE" H 7750 2250 50  0001 C CNN "PartNumber"
 	1    7750 2250
 	0    1    1    0
@@
 P 8000 2450
 F 0 "D5" V 7954 2529 50  0000 L CNN
-F 1 "3v3Zener" V 8045 2529 50  0000 L CNN
+F 1 "3.9V" V 8045 2529 50  0000 L CNN
 F 2 "Diode_SMD:D_SOD-323" H 8000 2450 50  0001 C CNN
 F 3 "~" H 8000 2450 50  0001 C CNN
+F 4 "C353523" H 8000 2450 50  0001 C CNN "LCSC"
+F 5 "BZT52C3V9S" H 8000 2450 50  0001 C CNN "PartNumber"
 	1    8000 2450
 	0    1    1    0
@@
 P 7750 3150
 F 0 "R18" V 7545 3150 50  0000 C CNN
-F 1 "1.8k" V 7636 3150 50  0000 C CNN
+F 1 "2.0k" V 7636 3150 50  0000 C CNN
 F 2 "Resistor_SMD:R_0402_1005Metric" V 7790 3140 50  0001 C CNN
 F 3 "~" H 7750 3150 50  0001 C CNN
+F 4 "C4109" H 7750 3150 50  0001 C CNN "LCSC"
+F 5 "0402WGF2001TCE" H 7750 3150 50  0001 C CNN "PartNumber"
 	1    7750 3150
 	0    1    1    0
@@
 P 8000 3350
 F 0 "D6" V 7954 3429 50  0000 L CNN
-F 1 "3v3Zener" V 8045 3429 50  0000 L CNN
+F 1 "3.9V" V 8045 3429 50  0000 L CNN
 F 2 "Diode_SMD:D_SOD-323" H 8000 3350 50  0001 C CNN
 F 3 "~" H 8000 3350 50  0001 C CNN
+F 4 "C353523" H 8000 3350 50  0001 C CNN "LCSC"
+F 5 "BZT52C3V9S" H 8000 3350 50  0001 C CNN "PartNumber"
 	1    8000 3350
 	0    1    1    0
@@
 P 7750 4050
 F 0 "R19" V 7545 4050 50  0000 C CNN
-F 1 "1.8k" V 7636 4050 50  0000 C CNN
+F 1 "2.0k" V 7636 4050 50  0000 C CNN
 F 2 "Resistor_SMD:R_0402_1005Metric" V 7790 4040 50  0001 C CNN
 F 3 "~" H 7750 4050 50  0001 C CNN
+F 4 "C4109" H 7750 4050 50  0001 C CNN "LCSC"
+F 5 "0402WGF2001TCE" H 7750 4050 50  0001 C CNN "PartNumber"
 	1    7750 4050
 	0    1    1    0
@@
 P 8000 4250
 F 0 "D7" V 7954 4329 50  0000 L CNN
-F 1 "3v3Zener" V 8045 4329 50  0000 L CNN
+F 1 "3.9V" V 8045 4329 50  0000 L CNN
 F 2 "Diode_SMD:D_SOD-323" H 8000 4250 50  0001 C CNN
 F 3 "~" H 8000 4250 50  0001 C CNN
+F 4 "C353523" H 8000 4250 50  0001 C CNN "LCSC"
+F 5 "BZT52C3V9S" H 8000 4250 50  0001 C CNN "PartNumber"
 	1    8000 4250
 	0    1    1    0
@@
 F 2 "Capacitor_SMD:C_0402_1005Metric" H 2288 2850 50  0001 C CNN
 F 3 "~" H 2250 3000 50  0001 C CNN
+F 4 "C1525" H 2250 3000 50  0001 C CNN "LCSC"
+F 5 "CL05B104KO5NNNC" H 2250 3000 50  0001 C CNN "PartNumber"
 	1    2250 3000
 	0    1    1    0
