File: Hardware/KiCAD/LuminaryVer1/PowerSupply.sch (KiCad schematic (older format))
At the start: 28 parts, among them Q1 2N3904, SW2 SW_BATT_DISCONNECT, U3 DIO6605, U4 AP2112K-3.3, U7 DW01, U8 FS8205A, U9 TP4056

Commit message: Routed entire power section
Parts:
- removed C12, C8: 1uF, Capacitor_SMD:C_0805_2012Metric, symbol Device:C_Small
- removed C14: 10uF, Capacitor_SMD:C_0805_2012Metric, symbol Device:C_Small
- R30: value 100 -> 120
Changed lines of the file:
@@
-$EndComp
-$Comp
-L Device:C_Small C8
-U 1 1 5E7A3834
-P 9150 3600
-F 0 "C8" H 9242 3646 50  0000 L CNN
-F 1 "1uF" H 9242 3555 50  0000 L CNN
-F 2 "Capacitor_SMD:C_0805_2012Metric" H 9150 3600 50  0001 C CNN
-F 3 "~" H 9150 3600 50  0001 C CNN
-	1    9150 3600
-	1    0    0    -1
 $EndComp
 $Comp
@@
 $EndComp
 Wire Wire Line
-	9150 3500 9150 3400
-Wire Wire Line
-	9150 3400 9350 3400
-Wire Wire Line
 	9450 3500 9350 3500
 Wire Wire Line
@@
 Wire Wire Line
 	10200 3400 10200 3500
-Wire Wire Line
-	9150 3700 9150 3900
-Wire Wire Line
-	9150 3900 9750 3900
 Wire Wire Line
 	9750 3900 9750 3800
@@
 Connection ~ 8750 3400
 Wire Wire Line
-	8750 3400 9150 3400
-Connection ~ 9150 3400
-Wire Wire Line
 	8750 3400 8750 3500
 Wire Wire Line
-	8750 3900 9150 3900
-Wire Wire Line
 	8750 3700 8750 3900
-Connection ~ 9150 3900
 $Comp
 L Device:D_Schottky D1
@@
 NoConn ~ 2150 5600
 $Comp
-L Device:C_Small C12
-U 1 1 5EB5FBF0
-P 3400 4300
-F 0 "C12" H 3492 4346 50  0000 L CNN
-F 1 "1uF" H 3492 4255 50  0000 L CNN
-F 2 "Capacitor_SMD:C_0805_2012Metric" H 3400 4300 50  0001 C CNN
-F 3 "~" H 3400 4300 50  0001 C CNN
-	1    3400 4300
-	1    0    0    -1
-$EndComp
-$Comp
 L Device:C_Small C13
 U 1 1 5EB609C6
@@
 	3750 4200 3750 4100
 Wire Wire Line
-	3750 4100 3400 4100
-Wire Wire Line
-	3400 4200 3400 4100
-Connection ~ 3400 4100
-Wire Wire Line
-	3400 4100 3250 4100
-Wire Wire Line
 	3300 4550 3300 4300
 Wire Wire Line
 	3300 4300 3250 4300
-Wire Wire Line
-	3400 4400 3400 4550
 Connection ~ 3400 4550
 Wire Wire Line
@@
 P 4000 4100
 F 0 "R30" V 4200 4100 50  0000 C CNN
-F 1 "100" V 4100 4100 50  0000 C CNN
+F 1 "120" V 4100 4100 50  0000 C CNN
 F 2 "Resistor_SMD:R_0402_1005Metric" V 4040 4090 50  0001 C CNN
 F 3 "~" H 4000 4100 50  0001 C CNN
@@
 Wire Wire Line
 	3950 2350 3950 2450
-$Comp
-L Device:C_Small C14
-U 1 1 5EBA06A5
-P 4050 2100
-F 0 "C14" H 3959 2054 50  0000 R CNN
-F 1 "10uF" H 3959 2145 50  0000 R CNN
-F 2 "Capacitor_SMD:C_0805_2012Metric" H 4050 2100 50  0001 C CNN
-F 3 "~" H 4050 2100 50  0001 C CNN
-	1    4050 2100
-	1    0    0    1
-$EndComp
-Wire Wire Line
-	4050 2000 4050 1950
-Wire Wire Line
-	4050 1950 3850 1950
-Wire Wire Line
-	4050 2200 4050 2250
 Wire Wire Line
 	4050 2850 3950 2850
 Connection ~ 3950 2850
-Wire Wire Line
-	4250 1950 4050 1950
-Connection ~ 4050 1950
 Text HLabel 1050 1950 0    50   UnSpc ~ 0
 Ext_In+
@@
 Wire Wire Line
 	3850 2250 4050 2250
-Connection ~ 4050 2250
 Wire Wire Line
 	4050 2250 4050 2850
@@
 Wire Wire Line
 	1900 4950 1900 5400
+Wire Wire Line
+	3250 4100 3750 4100
+Wire Wire Line
+	3850 1950 4250 1950
+Wire Wire Line
+	8750 3400 9350 3400
+Wire Wire Line
+	8750 3900 9750 3900
 $EndSCHEMATC

Commit message: Finalized for version 1 production.
Parts:
- C11, C13: footprint Capacitor_SMD:C_0805_2012Metric -> Capacitor_SMD:C_0402_1005Metric; LCSC (none) -> C1525; PartNumber (none) -> CL05B104KO5NNNC
- C6, C7: LCSC (none) -> C162316; PartNumber (none) -> GRM21BB31A106KE18L
- C9: LCSC (none) -> C28323; PartNumber (none) -> CL21B105KBFNNNE
- D1: LCSC (none) -> C266798; PartNumber (none) -> SS16HE3_B/H
- D8: LCSC (none) -> C205446; PartNumber (none) -> ORH-R36G
- D9: LCSC (none) -> C193191; PartNumber (none) -> ORH-B36G
- L1: value 4.3uH -> 3.3uH; LCSC (none) -> C315723; PartNumber CKP20164R7M-T -> MIP20124R7MBE
- Q1: LCSC (none) -> C18536; PartNumber (none) -> 2N3904S-RTK/PS
- R10, R31: value 50k -> 47k; LCSC (none) -> C25792; PartNumber (none) -> 0402WGF4702TCE
- R26, R27, R28: LCSC (none) -> C11702; PartNumber (none) -> 0402WGF1001TCE
- R29, R9: LCSC (none) -> C102759; PartNumber (none) -> RTT02103JTH
- R30: LCSC (none) -> C25079; PartNumber (none) -> 0402WGF1200TCE
- R8: LCSC (none) -> C325391; PartNumber (none) -> RMC04021005%N
- SW2: LCSC (none) -> C136659; PartNumber (none) -> K3-1296S-E2
- U3: Mouser (none) -> 453-DIO6605BFN8; PartNumber (none) -> DIO6605BFN8
- U4: LCSC (none) -> C51118; PartNumber (none) -> AP2112K-3.3TRG1
- U7: LCSC (none) -> C61503; PartNumber (none) -> DW01A-G
- U8: LCSC (none) -> C16052; PartNumber (none) -> FS8205A
- U9: LCSC (none) -> C382139; PartNumber (none) -> TP4056
Changed lines of the file:
@@
 F 2 "Package_TO_SOT_SMD:SOT-23-5" H 9750 3825 50  0001 C CNN
 F 3 "https://www.diodes.com/assets/Datasheets/AP2112.pdf" H 9750 3600 50  0001 C CNN
+F 4 "C51118" H 9750 3500 50  0001 C CNN "LCSC"
+F 5 "AP2112K-3.3TRG1" H 9750 3500 50  0001 C CNN "PartNumber"
 	1    9750 3500
 	1    0    0    -1
@@
 F 2 "Capacitor_SMD:C_0805_2012Metric" H 10200 3600 50  0001 C CNN
 F 3 "~" H 10200 3600 50  0001 C CNN
+F 4 "C28323" H 10200 3600 50  0001 C CNN "LCSC"
+F 5 "CL21B105KBFNNNE" H 10200 3600 50  0001 C CNN "PartNumber"
 	1    10200 3600
 	1    0    0    -1
@@
 F 2 "Package_DFN_QFN:DFN-8-1EP_2x3mm_P0.5mm_EP0.61x2.2mm" H 7700 3500 50  0001 C CNN
 F 3 "" H 7700 3500 50  0001 C CNN
+F 4 "453-DIO6605BFN8" H 7700 3350 50  0001 C CNN "Mouser"
+F 5 "DIO6605BFN8" H 7700 3350 50  0001 C CNN "PartNumber"
 	1    7700 3350
 	1    0    0    -1
@@
 P 7700 2900
 F 0 "L1" V 7981 2900 50  0000 C CNN
-F 1 "4.3uH" V 7890 2900 50  0000 C CNN
+F 1 "3.3uH" V 7890 2900 50  0000 C CNN
 F 2 "Inductor_SMD:L_0805_2012Metric" H 7700 2900 50  0001 C CNN
 F 3 "~" H 7700 2900 50  0001 C CNN
-F 4 "CKP20164R7M-T" V 7799 2900 50  0000 C CNN "PartNumber"
+F 4 "MIP20124R7MBE" V 7799 2900 50  0000 C CNN "PartNumber"
+F 5 "C315723" H 7700 2900 50  0001 C CNN "LCSC"
 	1    7700 2900
 	0    -1   -1   0
@@
 F 2 "Capacitor_SMD:C_0805_2012Metric" H 7000 3600 50  0001 C CNN
 F 3 "~" H 7000 3600 50  0001 C CNN
+F 4 "C162316" H 7000 3600 50  0001 C CNN "LCSC"
+F 5 "GRM21BB31A106KE18L" H 7000 3600 50  0001 C CNN "PartNumber"
 	1    7000 3600
 	1    0    0    1
@@
 F 2 "Capacitor_SMD:C_0805_2012Metric" H 8750 3600 50  0001 C CNN
 F 3 "~" H 8750 3600 50  0001 C CNN
+F 4 "C162316" H 8750 3600 50  0001 C CNN "LCSC"
+F 5 "GRM21BB31A106KE18L" H 8750 3600 50  0001 C CNN "PartNumber"
 	1    8750 3600
 	1    0    0    -1
@@
 F 2 "Diode_SMD:D_SMA" H 7550 4250 50  0001 C CNN
 F 3 "~" H 7550 4250 50  0001 C CNN
+F 4 "C266798" H 7550 4250 50  0001 C CNN "LCSC"
+F 5 "SS16HE3_B/H" H 7550 4250 50  0001 C CNN "PartNumber"
 	1    7550 4250
 	-1   0    0    1
@@
 P 8300 3500
 F 0 "R10" V 8500 3500 50  0000 C CNN
-F 1 "50k" V 8400 3500 50  0000 C CNN
+F 1 "47k" V 8400 3500 50  0000 C CNN
 F 2 "Resistor_SMD:R_0402_1005Metric" V 8340 3490 50  0001 C CNN
 F 3 "~" H 8300 3500 50  0001 C CNN
+F 4 "C25792" H 8300 3500 50  0001 C CNN "LCSC"
+F 5 "0402WGF4702TCE" H 8300 3500 50  0001 C CNN "PartNumber"
 	1    8300 3500
 	0    1    1    0
@@
 F 2 "Package_TO_SOT_SMD:SOT-23" H 8200 4475 50  0001 L CIN
 F 3 "https://www.fairchildsemi.com/datasheets/2N/2N3904.pdf" H 8000 4550 50  0001 L CNN
+F 4 "C18536" H 8000 4550 50  0001 C CNN "LCSC"
+F 5 "2N3904S-RTK/PS" H 8000 4550 50  0001 C CNN "PartNumber"
 	1    8000 4550
 	1    0    0    -1
@@
 F 2 "Resistor_SMD:R_0402_1005Metric" V 7590 4540 50  0001 C CNN
 F 3 "~" H 7550 4550 50  0001 C CNN
+F 4 "C325391" H 7550 4550 50  0001 C CNN "LCSC"
+F 5 "RMC04021005%N" H 7550 4550 50  0001 C CNN "PartNumber"
 	1    7550 4550
 	0    1    1    0
@@
 F 2 "Resistor_SMD:R_0402_1005Metric" V 7790 4790 50  0001 C CNN
 F 3 "~" H 7750 4800 50  0001 C CNN
+F 4 "C102759" H 7750 4800 50  0001 C CNN "LCSC"
+F 5 "RTT02103JTH" H 7750 4800 50  0001 C CNN "PartNumber"
 	1    7750 4800
 	-1   0    0    1
@@
 F 2 "Package_SO:TSSOP-8_4.4x3mm_P0.65mm" H 3700 5650 60  0001 C CNN
 F 3 "" H 3700 5650 60  0001 C CNN
+F 4 "C16052" H 2750 5400 50  0001 C CNN "LCSC"
+F 5 "FS8205A" H 2750 5400 50  0001 C CNN "PartNumber"
 	1    2750 5400
 	0    1    1    0
@@
 F 2 "PMIC:TP4056_SOP-8-PP" H 3350 2200 60  0001 C CNN
 F 3 "" H 3350 2200 60  0000 C CNN
+F 4 "C382139" H 3350 2200 50  0001 C CNN "LCSC"
+F 5 "TP4056" H 3350 2200 50  0001 C CNN "PartNumber"
 	1    3350 2200
 	1    0    0    -1
@@
 F 2 "Package_TO_SOT_SMD:SOT-23-6" H 2600 3950 60  0001 C CNN
 F 3 "" H 2600 3950 60  0001 C CNN
+F 4 "C61503" H 2650 4250 50  0001 C CNN "LCSC"
+F 5 "DW01A-G" H 2650 4250 50  0001 C CNN "PartNumber"
 	1    2650 4250
 	1    0    0    -1
@@
 F 0 "C13" H 3842 4346 50  0000 L CNN
 F 1 "100nF" H 3842 4255 50  0000 L CNN
-F 2 "Capacitor_SMD:C_0805_2012Metric" H 3750 4300 50  0001 C CNN
+F 2 "Capacitor_SMD:C_0402_1005Metric" H 3750 4300 50  0001 C CNN
 F 3 "~" H 3750 4300 50  0001 C CNN
+F 4 "C1525" H 3750 4300 50  0001 C CNN "LCSC"
+F 5 "CL05B104KO5NNNC" H 3750 4300 50  0001 C CNN "PartNumber"
 	1    3750 4300
 	1    0    0    -1
@@
 F 2 "Resistor_SMD:R_0402_1005Metric" V 4040 4090 50  0001 C CNN
 F 3 "~" H 4000 4100 50  0001 C CNN
+F 4 "C25079" H 4000 4100 50  0001 C CNN "LCSC"
+F 5 "0402WGF1200TCE" H 4000 4100 50  0001 C CNN "PartNumber"
 	1    4000 4100
 	0    1    -1   0
@@
 F 2 "Resistor_SMD:R_0402_1005Metric" V 3990 2590 50  0001 C CNN
 F 3 "~" H 3950 2600 50  0001 C CNN
+F 4 "C102759" H 3950 2600 50  0001 C CNN "LCSC"
+F 5 "RTT02103JTH" H 3950 2600 50  0001 C CNN "PartNumber"
 	1    3950 2600
 	-1   0    0    -1
@@
 F 2 "Diode_SMD:D_0603_1608Metric" H 2050 2150 50  0001 C CNN
 F 3 "~" H 2050 2150 50  0001 C CNN
+F 4 "C205446" H 2050 2150 50  0001 C CNN "LCSC"
+F 5 "ORH-R36G" H 2050 2150 50  0001 C CNN "PartNumber"
 	1    2050 2150
 	-1   0    0    1
@@
 F 2 "Diode_SMD:D_0603_1608Metric" H 2050 2450 50  0001 C CNN
 F 3 "~" H 2050 2450 50  0001 C CNN
+F 4 "C193191" H 2050 2450 50  0001 C CNN "LCSC"
+F 5 "ORH-B36G" H 2050 2450 50  0001 C CNN "PartNumber"
 	1    2050 2450
 	-1   0    0    1
@@
 F 2 "Resistor_SMD:R_0402_1005Metric" V 2490 2140 50  0001 C CNN
 F 3 "~" H 2450 2150 50  0001 C CNN
+F 4 "C11702" H 2450 2150 50  0001 C CNN "LCSC"
+F 5 "0402WGF1001TCE" H 2450 2150 50  0001 C CNN "PartNumber"
 	1    2450 2150
 	0    1    -1   0
@@
 F 2 "Resistor_SMD:R_0402_1005Metric" V 2490 2440 50  0001 C CNN
 F 3 "~" H 2450 2450 50  0001 C CNN
+F 4 "C11702" H 2450 2450 50  0001 C CNN "LCSC"
+F 5 "0402WGF1001TCE" H 2450 2450 50  0001 C CNN "PartNumber"
 	1    2450 2450
 	0    1    -1   0
@@
 F 0 "C11" H 1442 2346 50  0000 L CNN
 F 1 "100nF" H 1442 2255 50  0000 L CNN
-F 2 "Capacitor_SMD:C_0805_2012Metric" H 1350 2300 50  0001 C CNN
+F 2 "Capacitor_SMD:C_0402_1005Metric" H 1350 2300 50  0001 C CNN
 F 3 "~" H 1350 2300 50  0001 C CNN
+F 4 "C1525" H 1350 2300 50  0001 C CNN "LCSC"
+F 5 "CL05B104KO5NNNC" H 1350 2300 50  0001 C CNN "PartNumber"
 	1    1350 2300
 	-1   0    0    -1
@@
 F 2 "toggle:LCSC_C136659_HRO_SPDT_6.7x2.6mm_ToggleSwitch" H 6450 3200 50  0001 C CNN
 F 3 "~" H 6450 3200 50  0001 C CNN
+F 4 "C136659" H 6450 3200 50  0001 C CNN "LCSC"
+F 5 "K3-1296S-E2" H 6450 3200 50  0001 C CNN "PartNumber"
 	1    6450 3200
 	-1   0    0    -1
@@
 P 1650 2500
 F 0 "R31" V 1850 2500 50  0000 C CNN
-F 1 "50k" V 1750 2500 50  0000 C CNN
+F 1 "47k" V 1750 2500 50  0000 C CNN
 F 2 "Resistor_SMD:R_0402_1005Metric" V 1690 2490 50  0001 C CNN
 F 3 "~" H 1650 2500 50  0001 C CNN
+F 4 "C25792" H 1650 2500 50  0001 C CNN "LCSC"
+F 5 "0402WGF4702TCE" H 1650 2500 50  0001 C CNN "PartNumber"
 	1    1650 2500
 	-1   0    0    1
@@
 F 2 "Resistor_SMD:R_0402_1005Metric" V 1940 4790 50  0001 C CNN
 F 3 "~" H 1900 4800 50  0001 C CNN
+F 4 "C11702" H 1900 4800 50  0001 C CNN "LCSC"
+F 5 "0402WGF1001TCE" H 1900 4800 50  0001 C CNN "PartNumber"
 	1    1900 4800
 	-1   0    0    -1
