File: Hardware/KiCAD/LuminaryVer2/OutputDrive.sch (KiCad schematic (older format))
At the start: 16 parts, among them U5 SN65HVD232

Commit message: Updated version 2 hardware schematics.
Parts:
- removed D2, D3, D4, D5, D6, D7: 3.9V, Diode_SMD:D_SOD-323, symbol Device:D_Zener
- removed R14, R15, R16, R17, R18, R19: 2.0k, Resistor_SMD:R_0402_1005Metric, symbol Device:R_US
- removed R_PWR_2: 0, Resistor_SMD:R_0402_1005Metric, symbol Device:R_US
Connections:
- wire segments 52 -> 25
Other:
- note added: "(Originally buffered)"
- note added: "CAN Transciever"
- note added: "GPIO Passthrough"
- moved on the sheet: C10, R12, U5
