File: Hardware/KiCAD/LuminaryVer2/InputConnectors.sch (KiCad schematic (older format))
At the start: 13 parts, among them J1 JTAG, J10 ExtBattPwr, J12 USB_B_Micro, J2 GPIOInput, U1 74HC14

Commit message: Updated version 2 hardware schematics.
Parts:
- removed R_PWR_1: 0, Resistor_SMD:R_0402_1005Metric, symbol Device:R_US
- U1: footprint Package_SO:TSSOP-14_4.4x5mm_P0.65mm -> Package_SO:SOIC-14_3.9x8.7mm_P1.27mm; LCSC C5606 -> C5605
- U1: footprint Package_SO:TSSOP-14_4.4x5mm_P0.65mm -> Package_SO:SOIC-14_3.9x8.7mm_P1.27mm; LCSC C5606 -> C5605; PartNumber 74HC14PW,118 -> 74HC14D,653
Connections:
- net 3.3V+: now also C5.2, R20.1, R21.1, R22.1, R23.1, R24.1, R25.1, U1.14 (VCC)
- net D-: now reaches J12.2 (D-)
- net D+: now reaches J12.3 (D+)
Other:
- note added: "External Battery"
- note added: "External GPIO Input"
- note added: "JTAG Connector"
- note added: "USB Connector"
- moved on the sheet: C5, J1, J10, J12, J2, R20, R21, R22, R23, R24, R25, U1A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

Commit message: Add silk screen overlay to pins. Redo GPIO input to use LCSC basic part.
Connections:
- net 3.3V+: no longer R20.1, R21.1, R22.1, R23.1, R24.1, R25.1
- net GND: now also R20.1, R21.1, R22.1, R23.1, R24.1, R25.1
Changed lines of the file:
@@
 	5400 1600 5550 1600
-Wire Wire Line
-	8450 1600 8450 2750
 Wire Wire Line
 	5550 1700 5550 1600
@@
 Wire Wire Line
 	5650 2100 5650 1600
-Connection ~ 5650 1600
-Wire Wire Line
-	5650 1600 8450 1600
 Wire Wire Line
 	5650 2400 5650 3150
@@
 Text Notes 1500 3500 0    50   ~ 0
 USB Connector
+$Comp
+L power:GND #PWR?
+U 1 1 5EE14089
+P 4850 1650
+F 0 "#PWR?" H 4850 1400 50  0001 C CNN
+F 1 "GND" H 4855 1477 50  0000 C CNN
+F 2 "" H 4850 1650 50  0001 C CNN
+F 3 "" H 4850 1650 50  0001 C CNN
+	1    4850 1650
+	1    0    0    -1
+$EndComp
+Wire Wire Line
+	4850 1650 4850 1600
+Wire Wire Line
+	4850 1600 5050 1600
+Connection ~ 5050 1600
 $EndSCHEMATC

Commit message: Finalized hardware 2.3
Connections:
- no-connect marks 0 -> 2
Changed lines of the file:
@@
 	4850 1600 5050 1600
 Connection ~ 5050 1600
+NoConn ~ 2500 4300
+NoConn ~ 2100 2550
 $EndSCHEMATC
