File: Hardware/KiCAD/LuminaryVer2/LuminaryVer2.kicad_pcb (KiCad board)
At the start: 4 copper layers, 25.7 x 50 mm, 76 parts, among them J1 JTAG, J10 ExtBattPwr, J12 USB_B_Micro, J13 CN1, J14 CN2, J2 GPIOInput, Q1 2N3904, SW1 SW_Push, SW2 SW_BATT_DISCONNECT, U1 74HC14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

Commit message: Luminary V2 complete & sent off for manufacturing
Routing:
- net GND: track 52.4 -> 51.8 mm
Other:
- rule pad_to_mask_clearance: -0.051 -> 0
Changed lines of the file:
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@@
     (thickness 1.6)
     (drawings 71)
-    (tracks 777)
+    (tracks 776)
     (zones 0)
     (modules 76)
@@
   (layers
     (0 F.Cu signal)
-    (1 In1.Cu signal)
+    (1 In1.Cu signal hide)
     (2 In2.Cu signal hide)
     (31 B.Cu signal)
@@
     (33 F.Adhes user hide)
     (34 B.Paste user)
-    (35 F.Paste user hide)
+    (35 F.Paste user)
     (36 B.SilkS user hide)
     (37 F.SilkS user)
     (38 B.Mask user)
-    (39 F.Mask user)
+    (39 F.Mask user hide)
     (40 Dwgs.User user hide)
     (41 Cmts.User user hide)
@@
     (pad_size 1.524 1.524)
     (pad_drill 0.762)
-    (pad_to_mask_clearance -0.051)
+    (pad_to_mask_clearance 0)
     (solder_mask_min_width 0.25)
-    (pad_to_paste_clearance_ratio -0.15)
     (aux_axis_origin 210.9 100)
     (grid_origin 210.9 100)
@@
   (segment (start 228.305 65.66) (end 229.548 65.66) (width 0.381) (layer F.Cu) (net 1))
   (segment (start 229.591 65.703) (end 229.784 65.51) (width 0.381) (layer F.Cu) (net 1))
-  (via (at 229.9 89.9) (size 0.45) (drill 0.2) (layers F.Cu B.Cu) (net 1))
-  (via (at 229.9 92.45) (size 0.45) (drill 0.2) (layers F.Cu B.Cu) (net 1))
-  (segment (start 229.9 92) (end 229.9 92.45) (width 0.25) (layer F.Cu) (net 1))
-  (segment (start 229.135 91.75) (end 229.65 91.75) (width 0.25) (layer F.Cu) (net 1))
-  (segment (start 229.65 91.75) (end 229.9 92) (width 0.25) (layer F.Cu) (net 1))
-  (segment (start 229.9 89.5) (end 229.9 89.9) (width 0.25) (layer F.Cu) (net 1))
-  (segment (start 229.185 89.25) (end 229.65 89.25) (width 0.25) (layer F.Cu) (net 1))
-  (segment (start 229.65 89.25) (end 229.9 89.5) (width 0.25) (layer F.Cu) (net 1))
   (segment (start 229.15 94.3) (end 229.65 94.3) (width 0.25) (layer F.Cu) (net 1))
   (segment (start 229.65 94.3) (end 229.9 94.55) (width 0.25) (layer F.Cu) (net 1))
@@
   (segment (start 224.2 82.85) (end 223.925003 82.575003) (width 0.635) (layer B.Cu) (net 1))
   (segment (start 225.726 82.982) (end 224.316 82.982) (width 0.635) (layer B.Cu) (net 1))
+  (segment (start 229.650006 89.25) (end 229.9 89.499994) (width 0.25) (layer F.Cu) (net 1))
+  (segment (start 229.185 89.25) (end 229.650006 89.25) (width 0.25) (layer F.Cu) (net 1))
+  (via (at 229.9 89.499994) (size 0.45) (drill 0.2) (layers F.Cu B.Cu) (net 1))
+  (via (at 229.9 92.2) (size 0.45) (drill 0.2) (layers F.Cu B.Cu) (net 1))
+  (segment (start 229.9 91.85) (end 229.9 92.2) (width 0.25) (layer F.Cu) (net 1))
+  (segment (start 229.135 91.75) (end 229.8 91.75) (width 0.25) (layer F.Cu) (net 1))
+  (segment (start 229.8 91.75) (end 229.9 91.85) (width 0.25) (layer F.Cu) (net 1))
   (via (at 217.45 64.15) (size 0.45) (drill 0.2) (layers F.Cu B.Cu) (net 2))
   (via (at 218.45 64.15) (size 0.45) (drill 0.2) (layers F.Cu B.Cu) (net 2))
@@
   (segment (start 225.95 54.45) (end 225.95 54.881155) (width 0.25) (layer F.Cu) (net 67))
   (segment (start 231.615 53.4) (end 231.615 54.4) (width 0.508) (layer F.Cu) (net 67))
-  (segment (start 229.17 90.5) (end 229.85 90.5) (width 0.25) (layer F.Cu) (net 68))
-  (segment (start 232.77 93.42) (end 235.1 93.42) (width 0.25) (layer F.Cu) (net 68))
-  (segment (start 229.85 90.5) (end 229.8875 90.5375) (width 0.25) (layer F.Cu) (net 68))
-  (segment (start 229.8875 90.5375) (end 232.77 93.42) (width 0.25) (layer F.Cu) (net 68))
-  (via (at 229.8875 90.5375) (size 0.45) (drill 0.2) (layers F.Cu B.Cu) (net 68))
-  (segment (start 229.8875 90.5375) (end 229.3375 90.5375) (width 0.254) (layer In1.Cu) (net 68))
-  (segment (start 229.125 81.593198) (end 229.125 81.275) (width 0.254) (layer In1.Cu) (net 68))
   (via (at 229.125 81.275) (size 0.45) (drill 0.2) (layers F.Cu B.Cu) (net 68))
-  (segment (start 229.3375 90.5375) (end 229.125 90.325) (width 0.254) (layer In1.Cu) (net 68))
-  (segment (start 229.125 90.325) (end 229.125 81.593198) (width 0.254) (layer In1.Cu) (net 68))
   (segment (start 227.249874 81.275) (end 229.125 81.275) (width 0.254) (layer F.Cu) (net 68))
   (segment (start 226.66101 81.863864) (end 227.249874 81.275) (width 0.254) (layer F.Cu) (net 68))
+  (segment (start 229.17 90.5) (end 229.670473 90.5) (width 0.25) (layer F.Cu) (net 68))
+  (segment (start 232.590473 93.42) (end 230.078838 90.908365) (width 0.25) (layer F.Cu) (net 68))
+  (segment (start 229.535641 90.683366) (end 229.853839 90.683366) (width 0.254) (layer In1.Cu) (net 68))
+  (segment (start 229.670473 90.5) (end 229.853839 90.683366) (width 0.25) (layer F.Cu) (net 68))
+  (segment (start 230.078838 90.908365) (end 229.853839 90.683366) (width 0.25) (layer F.Cu) (net 68))
+  (via (at 229.853839 90.683366) (size 0.45) (drill 0.2) (layers F.Cu B.Cu) (net 68))
+  (segment (start 229.125 81.275) (end 229.125 90.272725) (width 0.254) (layer In1.Cu) (net 68))
+  (segment (start 229.125 90.272725) (end 229.535641 90.683366) (width 0.254) (layer In1.Cu) (net 68))
+  (segment (start 235.1 93.42) (end 232.590473 93.42) (width 0.25) (layer F.Cu) (net 68))
   (segment (start 229.135 93.05) (end 229.9 93.05) (width 0.25) (layer F.Cu) (net 69))
   (segment (start 233.66 95.96) (end 235.1 95.96) (width 0.25) (layer F.Cu) (net 69))
@@
     (polygon
       (pts
-        (xy 223.25 58.275) (xy 224.6 58.25) (xy 224.6 60.6) (xy 221.95 60.6) (xy 221.95 57.6)
-        (xy 217.95 57.6) (xy 217.55 58.05) (xy 217.55 61.65) (xy 216.95 62.25) (xy 214.5 62.25)
+        (xy 223.25 58.275) (xy 224.6 58.25) (xy 224.6 60.4) (xy 221.95 60.4) (xy 221.95 57.6)
+        (xy 217.55 57.6) (xy 217.55 58.05) (xy 217.55 61.65) (xy 216.95 62.25) (xy 214.5 62.25)
         (xy 214.5 64.55) (xy 210.95 64.55) (xy 210.9 64.5) (xy 210.9 60.65) (xy 216.2 60.65)
         (xy 216.45 60.35) (xy 216.45 56.7) (xy 217.55 55.6) (xy 217.55 54.1) (xy 223.25 54.125)
@@
       (pts
         (xy 230.95 69.45) (xy 228.95 71.45) (xy 228.95 78.75) (xy 223.9 78.65) (xy 223.9 74.45)
-        (xy 228 74.5) (xy 228 70.9) (xy 228.6 70.375) (xy 228.6 68.225) (xy 230.95 68.2)
+        (xy 228.15 74.5) (xy 228.15 70.9) (xy 228.6 70.5) (xy 228.6 68.225) (xy 230.95 68.2)
       )
     )

Commit message: Finalized hardware 2.3
Parts:
- removed R10: 1k, Resistor_SMD:R_0402_1005Metric
- Q1: value 2N3904 -> MMBT3904
- moved R13 2.05 mm to (232.7, 63.1)
- moved Q1 0.61 mm to (231.2, 66.6), turned to 90 degrees
Connections:
- Q1 pad 1: GND -> Net-(Q1-Pad1)
- Q1 pad 2: Net-(Q1-Pad2) -> GND
- R13 pad 1: GND -> Net-(Q1-Pad3)
- R13 pad 2: Net-(Q1-Pad3) -> Net-(C6-Pad2)
- R8 pad 1: Net-(Q1-Pad2) -> Net-(Q1-Pad1)
- R9 pad 2: Net-(Q1-Pad2) -> Net-(Q1-Pad1)
Routing:
- net Net-(Q1-Pad1): track 0.00 -> 2.89 mm
- net Net-(Q1-Pad2): track 2.23 -> 0.00 mm
- net Net-(Q1-Pad3): track 5.15 -> 3.14 mm
- net GND: track 51.8 -> 53.1 mm
Other:
- board text added: "Cortex-M4 Low Power Dev Board STM32L432KBU6 Rev 2.1 https://github.com/brandonbraun653/Luminary"
- board text added: "Key"
