File: Hardware/KiCAD/LuminaryVer2/PowerSupply.sch (KiCad schematic (older format))
At the start: 25 parts, among them Q1 2N3904, SW2 SW_BATT_DISCONNECT, U3 DIO6605, U4 AP2112K-3.3, U7 DW01, U8 FS8205A, U9 TP4056

Commit message: Updated version 2 hardware schematics.
Parts:
- removed U3: DIO6605, Package_DFN_QFN:DFN-8-1EP_2x3mm_P0.5mm_EP0.61x2.2mm, symbol LuminaryVer1-rescue:DIO6605-BoostConverters
- removed U4: AP2112K-3.3, Package_TO_SOT_SMD:SOT-23-5, symbol Regulator_Linear:AP2112K-3.3
- added C8: 10uF, Capacitor_SMD:C_0805_2012Metric, symbol Device:C_Small
- added D2: SS14, Diode_SMD:D_SMA, symbol Device:D_Schottky
- added R13: 10k, Resistor_SMD:R_0402_1005Metric, symbol Device:R_US
- added R14: 200k, Resistor_SMD:R_0603_1608Metric, symbol Device:R_US
- added R15: 620k, Resistor_SMD:R_0603_1608Metric, symbol Device:R_US
- added U3: TPS61040, Package_TO_SOT_SMD:SOT-23-5, symbol Regulator_Switching:TPS61041DDC
- added U4: AMS1117-3.3, Package_TO_SOT_SMD:SOT-223-3_TabPin2, symbol Regulator_Linear:AMS1117-3.3
- C6: LCSC C162316 -> C15850
- C7: value 10uF -> 3.3pF; footprint Capacitor_SMD:C_0805_2012Metric -> Capacitor_SMD:C_0402_1005Metric; LCSC C162316 -> C1565; PartNumber GRM21BB31A106KE18L -> CL05B104KO5NNNC
- D1: value SS16HE -> SS14; LCSC C266798 -> C2480
- D8: LCSC C205446 -> C2286; PartNumber ORH-R36G -> KT-0603R
- D9: LCSC C193191 -> C72041; PartNumber ORH-B36G -> 19-217/BHC-ZL1M2RY/3T
- R10: value 47k -> 1k; LCSC C25792 -> C11702
- R29, R9: LCSC C102759 -> C25744
- U7: value DW01 -> DW01+G; LCSC C61503 -> C14213
- U9: LCSC C382139 -> C16581
Connections:
- wire segments 126 -> 138
Other:
- note added: "Battery Charger"
- note added: "Battery Overvoltage Protection"
- note added: "Power Supply Generation"
- moved on the sheet: C11, C13, C6, C9, D1, D8, D9, L1, Q1, R10, R26, R27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

Commit message: Laid out the power supply updates.
Parts:
- added D5: BLED, Diode_SMD:D_0603_1608Metric, symbol Device:LED
- added R19: 1k, Resistor_SMD:R_0402_1005Metric, symbol Device:R_US
Connections:
- net Ext_In+: now also D5.2 (A)
- net GND: now also R19.1
- new net: D5.1 (K), R19.2
Changed lines of the file:
@@
 	7350 5550 7350 5650
 Wire Wire Line
-	5900 4750 6450 4750
+	5900 4750 6250 4750
 Wire Wire Line
 	6650 5050 6450 5050
@@
 	6050 5000 6050 5550
 Wire Wire Line
-	6050 5550 7000 5550
+	6050 5550 6250 5550
 Connection ~ 7000 5550
 Wire Wire Line
 	5900 4900 6050 4900
-Wire Wire Line
-	6050 4900 6050 5000
 Connection ~ 6050 5000
 $Comp
@@
 Text Notes 5500 3000 0    50   ~ 0
 Power Supply Generation
+$Comp
+L Device:LED D5
+U 1 1 5EE5242B
+P 6250 4950
+F 0 "D5" H 6400 4900 50  0000 C CNN
+F 1 "BLED" H 6250 5050 50  0000 C CNN
+F 2 "Diode_SMD:D_0603_1608Metric" H 6250 4950 50  0001 C CNN
+F 3 "~" H 6250 4950 50  0001 C CNN
+F 4 "C72041" H 6250 4950 50  0001 C CNN "LCSC"
+F 5 "19-217/BHC-ZL1M2RY/3T" H 6250 4950 50  0001 C CNN "PartNumber"
+	1    6250 4950
+	0    -1   -1   0
+$EndComp
+$Comp
+L Device:R_US R19
+U 1 1 5EE53684
+P 6250 5350
+F 0 "R19" V 6450 5350 50  0000 C CNN
+F 1 "1k" V 6350 5350 50  0000 C CNN
+F 2 "Resistor_SMD:R_0402_1005Metric" V 6290 5340 50  0001 C CNN
+F 3 "~" H 6250 5350 50  0001 C CNN
+F 4 "C11702" H 6250 5350 50  0001 C CNN "LCSC"
+F 5 "0402WGF1001TCE" H 6250 5350 50  0001 C CNN "PartNumber"
+	1    6250 5350
+	1    0    0    1
+$EndComp
+Wire Wire Line
+	6050 4900 6050 5000
+Wire Wire Line
+	6250 4800 6250 4750
+Connection ~ 6250 4750
+Wire Wire Line
+	6250 4750 6450 4750
+Wire Wire Line
+	6250 5100 6250 5200
+Wire Wire Line
+	6250 5500 6250 5550
+Connection ~ 6250 5550
+Wire Wire Line
+	6250 5550 7000 5550
 $EndSCHEMATC

Commit message: Luminary V2 complete & sent off for manufacturing
Parts:
- L1: LCSC C315723 -> C51725
- R8: LCSC C325391 -> C25076
Changed lines of the file:
@@
 F 3 "~" H 7700 3450 50  0001 C CNN
 F 4 "MIP20124R7MBE" V 7799 3450 50  0000 C CNN "PartNumber"
-F 5 "C315723" H 7700 3450 50  0001 C CNN "LCSC"
+F 5 "C51725" H 7700 3450 50  0001 C CNN "LCSC"
 	1    7700 3450
 	0    -1   -1   0
@@
 F 2 "Resistor_SMD:R_0402_1005Metric" V 6840 5040 50  0001 C CNN
 F 3 "~" H 6800 5050 50  0001 C CNN
-F 4 "C325391" H 6800 5050 50  0001 C CNN "LCSC"
+F 4 "C25076" H 6800 5050 50  0001 C CNN "LCSC"
 F 5 "RMC04021005%N" H 6800 5050 50  0001 C CNN "PartNumber"
 	1    6800 5050

Commit message: Document a hardware bug with the power supply in version two of Luminary.
Other:
- note added: "HW BUG:\nThe pullup/down resistors on pin 4 of the TPS61040\nneed to be swapped. Currently the priority is given \nto the battery for which power supply takes precedance."
Changed lines of the file:
@@
 Wire Wire Line
 	6250 5550 7000 5550
+Text Notes 6750 2800 0    50   ~ 0
+HW BUG:\nThe pullup/down resistors on pin 4 of the TPS61040\nneed to be swapped. Currently the priority is given \nto the battery for which power supply takes precedance.
 $EndSCHEMATC

Commit message: Finalized hardware 2.3
Parts:
- removed Q1: 2N3904, Package_TO_SOT_SMD:SOT-23, symbol Transistor_BJT:2N3904
- removed R10: 1k, Resistor_SMD:R_0402_1005Metric, symbol Device:R_US
- added Q1: MMBT3904, Package_TO_SOT_SMD:SOT-23, symbol Transistor_BJT:MMBT3904
Connections:
- net GND: now also Q1.2 (E); no longer R13.1
- net at C6.2, L1.1, SW2.2 (B)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: now also R13.2
- net at U3.4 (EN): now also R13.1, Q1.3 (C); no longer R13.2
- net at R8.1, R9.2: now also Q1.1 (B)
Other:
- note removed: "HW BUG:\nThe pullup/down resistors on pin 4 of the TPS61040\nneed to be swapped. Currently the priority is given \nto the battery for which power supply takes precedance."
- moved on the sheet: R13
Changed lines of the file:
@@
-$EndComp
-$Comp
-L Device:R_US R10
-U 1 1 5E7C8142
-P 7150 3650
-F 0 "R10" V 7350 3650 50  0000 C CNN
-F 1 "1k" V 7250 3650 50  0000 C CNN
-F 2 "Resistor_SMD:R_0402_1005Metric" V 7190 3640 50  0001 C CNN
-F 3 "~" H 7150 3650 50  0001 C CNN
-F 4 "C11702" H 7150 3650 50  0001 C CNN "LCSC"
-F 5 "0402WGF4702TCE" H 7150 3650 50  0001 C CNN "PartNumber"
-	1    7150 3650
-	-1   0    0    1
-$EndComp
-$Comp
-L Transistor_BJT:2N3904 Q1
-U 1 1 5E7D2C44
-P 7250 5050
-F 0 "Q1" H 7440 5096 50  0000 L CNN
-F 1 "2N3904" H 7440 5005 50  0000 L CNN
-F 2 "Package_TO_SOT_SMD:SOT-23" H 7450 4975 50  0001 L CIN
-F 3 "https://www.fairchildsemi.com/datasheets/2N/2N3904.pdf" H 7250 5050 50  0001 L CNN
-F 4 "C18536" H 7250 5050 50  0001 C CNN "LCSC"
-F 5 "2N3904S-RTK/PS" H 7250 5050 50  0001 C CNN "PartNumber"
-	1    7250 5050
-	1    0    0    -1
 $EndComp
 $Comp
@@
 	7700 4150 7700 4450
 Wire Wire Line
-	6800 4450 7150 4450
-Wire Wire Line
 	7350 4850 7350 3850
 Wire Wire Line
@@
 L Device:R_US R13
 U 1 1 5EEAD752
-P 7150 4050
-F 0 "R13" V 7350 4050 50  0000 C CNN
-F 1 "10k" V 7250 4050 50  0000 C CNN
-F 2 "Resistor_SMD:R_0402_1005Metric" V 7190 4040 50  0001 C CNN
-F 3 "~" H 7150 4050 50  0001 C CNN
-F 4 "C25744" H 7150 4050 50  0001 C CNN "LCSC"
-F 5 "0402WGF4702TCE" H 7150 4050 50  0001 C CNN "PartNumber"
-	1    7150 4050
+P 7150 3650
+F 0 "R13" V 7350 3650 50  0000 C CNN
+F 1 "10k" V 7250 3650 50  0000 C CNN
+F 2 "Resistor_SMD:R_0402_1005Metric" V 7190 3640 50  0001 C CNN
+F 3 "~" H 7150 3650 50  0001 C CNN
+F 4 "C25744" H 7150 3650 50  0001 C CNN "LCSC"
+F 5 "0402WGF4702TCE" H 7150 3650 50  0001 C CNN "PartNumber"
+	1    7150 3650
 	-1   0    0    1
 $EndComp
-Wire Wire Line
-	7150 4200 7150 4450
-Connection ~ 7150 4450
-Wire Wire Line
-	7150 4450 7700 4450
 Wire Wire Line
 	7350 3850 7150 3850
@@
 	7150 3850 7150 3800
 Connection ~ 7350 3850
-Wire Wire Line
-	7150 3900 7150 3850
-Connection ~ 7150 3850
 Wire Wire Line
 	6700 3450 6800 3450
@@
 Wire Wire Line
 	6250 5550 7000 5550
-Text Notes 6750 2800 0    50   ~ 0
-HW BUG:\nThe pullup/down resistors on pin 4 of the TPS61040\nneed to be swapped. Currently the priority is given \nto the battery for which power supply takes precedance.
+Wire Wire Line
+	6800 4450 7700 4450
+$Comp
+L Transistor_BJT:MMBT3904 Q1
+U 1 1 5F1A0B4C
+P 7250 5050
+F 0 "Q1" H 7441 5096 50  0000 L CNN
+F 1 "MMBT3904" H 7441 5005 50  0000 L CNN
+F 2 "Package_TO_SOT_SMD:SOT-23" H 7450 4975 50  0001 L CIN
+F 3 "https://www.fairchildsemi.com/datasheets/2N/2N3904.pdf" H 7250 5050 50  0001 L CNN
+F 4 "C20526" H 7250 5050 50  0001 C CNN "LCSC"
+	1    7250 5050
+	1    0    0    -1
+$EndComp
 $EndSCHEMATC
