File: Hardware/KiCAD/LightDriverShieldVer1/LightDriverShieldVer1.sch (KiCad schematic (older format))
At the start: 25 parts, among them J1 Conn_01x12, J2 Conn_01x12, J3 Conn_01x06, J4 Screw_Terminal_01x04, J5 ExtVCC, Q1 2N3904, Q2 Si2301, Q3 2N3904, Q4 2N3904, Q5 2N3904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

Commit message: Routed the shield for version 1
Parts:
- C1: value C_Small -> 1uF
Connections:
- net GND: now also SW1.1, SW1.2, SW1.3, SW1.4, SW1.5, SW1.6; no longer SW1.10, SW1.11, SW1.12, SW1.7, SW1.8, SW1.9
- net at J3.1 (Pin_1): now also SW1.12; no longer SW1.1
- net at J3.2 (Pin_2): now also SW1.11; no longer SW1.2
- net at J3.3 (Pin_3): now also SW1.10; no longer SW1.3
- net at J3.4 (Pin_4): now also SW1.9; no longer SW1.4
- net at J3.5 (Pin_5): now also SW1.8; no longer SW1.5
- net at J3.6 (Pin_6): now also SW1.7; no longer SW1.6
Other:
- moved on the sheet: J3
Changed lines of the file:
@@
 EESchema Schematic File Version 4
+LIBS:LightDriverShieldVer1-cache
 EELAYER 29 0
 EELAYER END
@@
 P 5650 1150
 F 0 "C1" H 5742 1196 50  0000 L CNN
-F 1 "C_Small" H 5742 1105 50  0000 L CNN
+F 1 "1uF" H 5742 1105 50  0000 L CNN
 F 2 "Capacitor_SMD:C_0402_1005Metric" H 5650 1150 50  0001 C CNN
 F 3 "~" H 5650 1150 50  0001 C CNN
@@
 L power:GND #PWR0104
 U 1 1 5EE609DB
-P 2300 5250
-F 0 "#PWR0104" H 2300 5000 50  0001 C CNN
-F 1 "GND" H 2305 5077 50  0000 C CNN
-F 2 "" H 2300 5250 50  0001 C CNN
-F 3 "" H 2300 5250 50  0001 C CNN
-	1    2300 5250
-	1    0    0    -1
-$EndComp
-Wire Wire Line
-	2250 4700 2300 4700
-Wire Wire Line
-	2300 4700 2300 4800
-Wire Wire Line
-	2250 5100 2300 5100
-Connection ~ 2300 5100
-Wire Wire Line
-	2300 5100 2300 5200
-Wire Wire Line
-	2250 5000 2300 5000
-Connection ~ 2300 5000
-Wire Wire Line
-	2300 5000 2300 5100
-Wire Wire Line
-	2250 4900 2300 4900
-Connection ~ 2300 4900
-Wire Wire Line
-	2300 4900 2300 5000
-Wire Wire Line
-	2250 4800 2300 4800
-Connection ~ 2300 4800
-Wire Wire Line
-	2300 4800 2300 4900
-Wire Wire Line
-	2250 5200 2300 5200
-Connection ~ 2300 5200
-Wire Wire Line
-	2300 5200 2300 5250
+P 1550 5300
+F 0 "#PWR0104" H 1550 5050 50  0001 C CNN
+F 1 "GND" H 1555 5127 50  0000 C CNN
+F 2 "" H 1550 5300 50  0001 C CNN
+F 3 "" H 1550 5300 50  0001 C CNN
+	1    1550 5300
+	1    0    0    -1
+$EndComp
 $Comp
 L power:+3.3V #PWR0105
@@
 L Connector_Generic:Conn_01x06 J3
 U 1 1 5EE6A8E5
-P 1300 4900
-F 0 "J3" H 1218 5317 50  0000 C CNN
-F 1 "Conn_01x06" H 1218 5226 50  0000 C CNN
-F 2 "Connector_PinSocket_2.54mm:PinSocket_1x06_P2.54mm_Vertical" H 1300 4900 50  0001 C CNN
-F 3 "~" H 1300 4900 50  0001 C CNN
-	1    1300 4900
-	-1   0    0    -1
-$EndComp
-Wire Wire Line
-	1500 4700 1650 4700
-Wire Wire Line
-	1500 4800 1650 4800
-Wire Wire Line
-	1500 4900 1650 4900
-Wire Wire Line
-	1500 5000 1650 5000
-Wire Wire Line
-	1500 5100 1650 5100
-Wire Wire Line
-	1500 5200 1650 5200
+P 2450 4900
+F 0 "J3" H 2368 5317 50  0000 C CNN
+F 1 "Conn_01x06" H 2368 5226 50  0000 C CNN
+F 2 "Connector_PinSocket_2.54mm:PinSocket_1x06_P2.54mm_Vertical" H 2450 4900 50  0001 C CNN
+F 3 "~" H 2450 4900 50  0001 C CNN
+	1    2450 4900
+	1    0    0    -1
+$EndComp
 Text GLabel 1700 2000 2    50   Input ~ 0
 OUT3
@@
 Wire Wire Line
 	9550 1750 9650 1750
+Wire Wire Line
+	1550 5300 1550 5200
+Wire Wire Line
+	1550 4700 1650 4700
+Wire Wire Line
+	1650 4800 1550 4800
+Connection ~ 1550 4800
+Wire Wire Line
+	1550 4800 1550 4700
+Wire Wire Line
+	1650 4900 1550 4900
+Connection ~ 1550 4900
+Wire Wire Line
+	1550 4900 1550 4800
+Wire Wire Line
+	1650 5000 1550 5000
+Connection ~ 1550 5000
+Wire Wire Line
+	1550 5000 1550 4900
+Wire Wire Line
+	1650 5100 1550 5100
+Connection ~ 1550 5100
+Wire Wire Line
+	1550 5100 1550 5000
+Wire Wire Line
+	1650 5200 1550 5200
+Connection ~ 1550 5200
+Wire Wire Line
+	1550 5200 1550 5100
 $EndSCHEMATC
