File: Hardware/KiCAD/LightDriverShieldVer1/LightDriverShieldVer1.sch (KiCad schematic (older format))
At the start: 25 parts, among them J1 Conn_01x12, J2 Conn_01x12, J3 Conn_01x06, J4 Screw_Terminal_01x04, J5 ExtVCC, Q1 2N3904, Q2 Si2301, Q3 2N3904, Q4 2N3904, Q5 2N3904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

Commit message: Rev the LightDriver board to version 2.
Other:
- note added: "HW Note:\nWhy is OUT3 tied to CH2 and OUT2 is tied to CH3?"
Changed lines of the file:
@@
 Text Notes 5700 850  0    50   ~ 0
 HW Bug 3:\nFootprint of Q1 has pins 1 & 2 swapped, leading \nto loss of control of the power switch.
+Text Notes 550  2850 0    50   ~ 0
+HW Note:\nWhy is OUT3 tied to CH2 and OUT2 is tied to CH3?
 $EndSCHEMATC
